File: RelatBoard/48VRelay/48VERelay/MCU.kicad_sch (KiCad schematic)
At the start: 5 parts, among them U2 ESP32-PICO-V3

Commit message: sys_update
Parts:
- removed U2: ESP32-PICO-V3, Package_DFN_QFN:QFN-48-1EP_7x7mm_P0.5mm_EP5.3x5.3mm, symbol MCU_Espressif:ESP32-PICO-V3
- added C11, C12, C13, C14, C15, C16, C7: 0.1uF, symbol Device:C_Small
- added C17, C19: 6.8nF, symbol Device:C_Small
- added C18: 10uF / 16V, symbol Device:C_Polarized_Small_US
- added C20, C23: 10nF, symbol Device:C_Small
- added C21, C22: 18pF, symbol Device:C_Small
- added C5: 4.7uF - Eth Reference Cap, symbol Device:C_Small
- added C6: 22nF, symbol Device:C_Small
- added C8: 10uF, symbol Device:C_Small
- added L1: MH1608-121Y, symbol Device:L_Ferrite_Small
- added R16, R17, R7, R8: 33, symbol Device:R_Small
- added R18, R19, R21, R22: 49.9 1%, symbol Device:R_Small
- added R20: 10 1%, symbol Device:R_Small
- added R23: 0, symbol Device:R_Small
- added R24: 1M, symbol Device:R_Small
- added R6: 12.4k 1% - Ethernet external reference, symbol Device:R_Small
- added U1: ESP32-WROOM-32UE, RF_Module:ESP32-WROOM-32UE, symbol RF_Module:ESP32-WROOM-32UE
- added U3: W5500, Package_QFP:LQFP-48_7x7mm_P0.5mm, symbol Interface_Ethernet:W5500
- added Y1: 25MHz, symbol Device:Crystal_GND3_Small
Connections:
- net GND: now also C11.2, C12.2, C13.2, C14.2, C15.2, C16.2, C18.2, C20.1, C21.2, C22.2, C23.2, C5.2, C6.2, C7.2, C8.2, R6.2, U1.[1,15,38,39] (GND), U3.14 (AGND), U3.16 (AGND), U3.19 (AGND), U3.29 (GND), U3.3 (AGND), U3.48 (AGND), U3.9 (AGND), Y1.3
- net +3V3 renamed +3V3 MCU
- net +3V3 MCU: now also U1.2 (VDD)
- new net: R16.1, U3.5 (RXN)
- new net: C17.1, R16.2, R21.1
- new net: C19.1, R17.2, R22.1
- new net: R7.1, U3.1 (TXN)
- new net: R6.1, U3.10 (EXRES1)
- new net: R23.1, R24.1, U3.31 (XO)
- new net: C21.1, R23.2, Y1.2
- new net: R8.1, U3.2 (TXP)
- new net: C5.1, U3.20 (TOCAP)
- new net: C23.1, U3.22 (1V2O)
- new net: C22.1, R24.2, U3.30 (XI/CLKIN), Y1.1
- new net: R17.1, U3.6 (RXP)
- new net +3V3 Eth: C7.1, C8.1, L1.1, U3.28 (VDD)
- new net +3V3A: C11.1, C12.1, C13.1, C14.1, C15.1, C16.1, C18.1, L1.2, R18.1, R19.1, R20.1, U3.11 (AVDD), U3.15 (AVDD), U3.17 (AVDD), U3.21 (AVDD), U3.4 (AVDD), U3.8 (AVDD)
- new net ACT LED: U3.27 (ACTLED)
- new net Ether_CS: U1.9 (IO33), U3.32 (~{SCS})
- new net Ether_INT: U1.12 (IO27), U3.36 (~{INT})
- new net Ether_MISO: U1.31 (IO19), U3.34 (MISO)
- new net Ether_MOSI: U1.37 (IO23), U3.35 (MOSI)
- new net Ether_RESET: U1.10 (IO25), U3.37 (~{RST})
- new net Ether_SCLK: U1.30 (IO18), U3.33 (SCLK)
- new net JTAG_RESET: U1.3 (EN)
- new net JTAG_TCK: U1.16 (IO13)
- new net JTAG_TDI: U1.14 (IO12)
- new net JTAG_TDO: U1.23 (IO15)
- new net JTAG_TMS: U1.13 (IO14)
- new net LINK LED: U3.25 (LINKLED)
- new net RELAY_1: U1.27 (IO16)
- new net RELAY_2: U1.28 (IO17)
- new net RELAY_3: U1.33 (IO21)
- new net RELAY_4: U1.36 (IO22)
- new net RELAY_5: U1.8 (IO32)
- new net RX_CT: C20.2, R21.2, R22.2
- new net RX_N: C17.2
- new net RX_P: C19.2
- new net TX_CT: C6.1, R20.2
- new net TX_N: R18.2, R7.2
- new net TX_P: R19.2, R8.2
Other:
- note added: "Keep trace short"
- note added: "Pulled up internally for auto-negoitation"

Commit message: begin pcb design
Parts:
- added D6: LED, LED_SMD:LED_0201_0603Metric, symbol Device:LED
- added R29: 330, Resistor_SMD:R_0603_1608Metric, symbol Device:R_Small
- C1, C18, C2, C5, C8: footprint (none) -> Capacitor_SMD:C_0805_2012Metric
- C11, C12, C13, C14, C15, C16, C17, C19, C21, C22, C23, C3, C4, C6, C7: footprint (none) -> Capacitor_SMD:C_0201_0603Metric
- R16, R17, R18, R20, R21, R22, R23, R24, R6, R7, R8: footprint (none) -> Resistor_SMD:R_0603_1608Metric
- R19: footprint (none) -> Resistor_SMD:R_0805_2012Metric
Connections:
- net +3V3 MCU: now also R29.1
- net GND: now also D6.1 (K)
- new net: D6.2 (A), R29.2
Other:
- note added: "PHY power"
- moved on the sheet: C11, C12, C13, C14, C15, C16, C17, C18, C19, C20, C21, C22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

Commit message: Begin PCB layout
Parts:
- removed Y1: 25MHz, symbol Device:Crystal_GND3_Small
- added J3: Conn_ARM_SWD_TagConnect_TC2030-NL, Connector:Tag-Connect_TC2030-IDC-NL_2x03_P1.27mm_Vertical, symbol Connector:Conn_ARM_SWD_TagConnect_TC2030-NL
- added Y2: ABM3C-25.000MHZ-D4Y-T, Library:CRYSTAL_ABM3C_ABR-M, symbol Crystal25MHz:ABM3C-25.000MHZ-D4Y-T
- C20: footprint (none) -> Capacitor_SMD:C_0201_0603Metric
- L1: footprint (none) -> Library:IND_BOURNS_MH1608
Connections:
- net GND: now also Y2.2, Y2.4
- net at C21.1, R23.2: now also Y2.1
- net at C22.1, R24.2, U3.30 (XI/CLKIN): now also Y2.3
- net RELAY_1 renamed MCU_RELAY_1
- net RELAY_2 renamed MCU_RELAY_2
- net RELAY_3 renamed MCU_RELAY_3
- net RELAY_4 renamed MCU_RELAY_4
- net RELAY_5 renamed MCU_RELAY_5
