File: RelatBoard/48VRelay/48VERelay/Outputs.kicad_sch (KiCad schematic)
At the start: 16 parts, among them J10 Screw_Terminal_01x03, J11 Screw_Terminal_01x03, J12 Screw_Terminal_01x03, J13 Screw_Terminal_01x03, J14 Screw_Terminal_01x03, K10 G2RL-1-E, K11 G2RL-1-E, K12 G2RL-1-E, K13 G2RL-1-E, K14 G2RL-1-E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

Commit message: sys_update
Parts:
- added D1, D2, D3, D4, D5: LED VO-PT2012SEAC, symbol Device:LED
- added R1, R2, R3, R4, R5: 2.2k, symbol Device:R_Small
- added R10, R11, R12, R13, R14: 10k, symbol Device:R_Small
- renumbered U1 to U2
Connections:
- net GND: now also D1.1 (K), D2.1 (K), D3.1 (K), D4.1 (K), D5.1 (K), R10.2, R11.2, R12.2, R13.2, R14.2
- net Relay_1: now also R1.2
- net Relay_2: now also R2.2
- net Relay_3: now also R3.2
- net Relay_4: now also R5.2
- net Relay_5: now also R4.2
- net RELAY_5: now reaches U2.1 (I1)
- net RELAY_5: now also U2.2 (I2), U2.3 (I3), U2.5 (I5), R10.1, R12.1, R13.1, R14.1
- net RELAY_4: now reaches U2.4 (I4)
- net RELAY_4: now also R11.1
- new net: D2.2 (A), R2.1
- new net: D5.2 (A), R5.1
- new net: D4.2 (A), R4.1
- new net: D3.2 (A), R3.1
- new net: D1.2 (A), R1.1
Other:
- moved on the sheet: 0685T5000-01, 0685T5000-2, 0685T5000-3, 0685T5000-4, 0685T5000-5, J10, J11, J12, J13, J14, K10, U2

Commit message: begin pcb design
Parts:
- 0685T5000-2, 0685T5000-3, 0685T5000-4, 0685T5000-5: footprint (none) -> Fuse:Fuse_0603_1608Metric
- D1, D2, D3, D4, D5: footprint (none) -> LED_SMD:LED_0201_0603Metric
- R1, R10, R11, R12, R13, R14, R2, R3, R4, R5: footprint (none) -> Resistor_SMD:R_0603_1608Metric
Changed lines of the file:
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@@
 		(unit 1)
 		(body_style 1)
-		(exclude_from_sim no)
+		(exclude_from_sim yes)
 		(in_bom yes)
 		(on_board yes)
@@
 			)
 		)
-		(property "Footprint" ""
+		(property "Footprint" "Resistor_SMD:R_0603_1608Metric"
 			(at 129.54 66.04 0)
 			(hide yes)
@@
 			)
 		)
-		(property "Footprint" ""
+		(property "Footprint" "Fuse:Fuse_0603_1608Metric"
 			(at 222.25 121.92 0)
 			(hide yes)
@@
 			)
 		)
-		(property "Footprint" ""
+		(property "Footprint" "Resistor_SMD:R_0603_1608Metric"
 			(at 129.54 76.2 0)
 			(hide yes)
@@
 		(unit 1)
 		(body_style 1)
-		(exclude_from_sim no)
+		(exclude_from_sim yes)
 		(in_bom yes)
 		(on_board yes)
@@
 			)
 		)
-		(property "Footprint" ""
+		(property "Footprint" "Fuse:Fuse_0603_1608Metric"
 			(at 222.25 96.52 0)
 			(hide yes)
@@
 			)
 		)
-		(property "Footprint" ""
+		(property "Footprint" "Resistor_SMD:R_0603_1608Metric"
 			(at 77.47 78.74 0)
 			(hide yes)
@@
 			)
 		)
-		(property "Footprint" ""
+		(property "Footprint" "Fuse:Fuse_0603_1608Metric"
 			(at 222.25 71.12 0)
 			(hide yes)
@@
 			)
 		)
-		(property "Footprint" ""
+		(property "Footprint" "Fuse:Fuse_0603_1608Metric"
 			(at 222.25 147.32 0)
 			(hide yes)
@@
 			)
 		)
-		(property "Footprint" ""
+		(property "Footprint" "Resistor_SMD:R_0603_1608Metric"
 			(at 54.61 71.12 0)
 			(hide yes)
@@
 			)
 		)
-		(property "Footprint" ""
+		(property "Footprint" "LED_SMD:LED_0201_0603Metric"
 			(at 115.57 85.09 0)
 			(hide yes)
@@
 		(unit 1)
 		(body_style 1)
-		(exclude_from_sim no)
+		(exclude_from_sim yes)
 		(in_bom yes)
 		(on_board yes)
@@
 			)
 		)
-		(property "Footprint" ""
+		(property "Footprint" "Resistor_SMD:R_0603_1608Metric"
 			(at 144.78 68.58 0)
 			(hide yes)
@@
 			)
 		)
-		(property "Footprint" ""
+		(property "Footprint" "LED_SMD:LED_0201_0603Metric"
 			(at 129.54 59.69 0)
 			(hide yes)
@@
 			)
 		)
-		(property "Footprint" ""
+		(property "Footprint" "LED_SMD:LED_0201_0603Metric"
 			(at 129.54 82.55 0)
 			(hide yes)
@@
 		(instances
 			(project "48VERelay"
-				(path "/2d740e7a-a48e-41b8-b74e-ca0ab277f7d9"
-					(reference "#PWR06")
-					(unit 1)
-				)
 				(path "/2d740e7a-a48e-41b8-b74e-ca0ab277f7d9/9acca724-bbf8-479c-b765-a30537109626"
 					(reference "#PWR06")
@@
 			)
 		)
-		(property "Footprint" ""
+		(property "Footprint" "Resistor_SMD:R_0603_1608Metric"
 			(at 69.85 76.2 0)
 			(hide yes)
@@
 		(unit 1)
 		(body_style 1)
-		(exclude_from_sim no)
+		(exclude_from_sim yes)
 		(in_bom yes)
 		(on_board yes)
@@
 		(unit 1)
 		(body_style 1)
-		(exclude_from_sim no)
+		(exclude_from_sim yes)
 		(in_bom yes)
 		(on_board yes)
@@
 		(instances
 			(project "48VERelay"
-				(path "/2d740e7a-a48e-41b8-b74e-ca0ab277f7d9"
-					(reference "0685T5000-01")
-					(unit 1)
-				)
 				(path "/2d740e7a-a48e-41b8-b74e-ca0ab277f7d9/9acca724-bbf8-479c-b765-a30537109626"
 					(reference "0685T5000-01")
@@
 			)
 		)
-		(property "Footprint" ""
+		(property "Footprint" "Resistor_SMD:R_0603_1608Metric"
 			(at 115.57 63.5 0)
 			(hide yes)
@@
 			)
 		)
-		(property "Footprint" ""
+		(property "Footprint" "Resistor_SMD:R_0603_1608Metric"
 			(at 115.57 78.74 0)
 			(hide yes)
@@
 		(instances
 			(project "48VERelay"
-				(path "/2d740e7a-a48e-41b8-b74e-ca0ab277f7d9"
-					(reference "#PWR01")
-					(unit 1)
-				)
 				(path "/2d740e7a-a48e-41b8-b74e-ca0ab277f7d9/9acca724-bbf8-479c-b765-a30537109626"
 					(reference "#PWR01")
@@
 			)
 		)
-		(property "Footprint" ""
+		(property "Footprint" "Resistor_SMD:R_0603_1608Metric"
 			(at 46.99 68.58 0)
 			(hide yes)
@@
 			)
 		)
-		(property "Footprint" ""
+		(property "Footprint" "Resistor_SMD:R_0603_1608Metric"
 			(at 62.23 73.66 0)
 			(hide yes)
@@
 			)
 		)
-		(property "Footprint" ""
+		(property "Footprint" "LED_SMD:LED_0201_0603Metric"
 			(at 144.78 62.23 0)
 			(hide yes)
@@
 			)
 		)
-		(property "Footprint" ""
+		(property "Footprint" "LED_SMD:LED_0201_0603Metric"
 			(at 115.57 57.15 0)
 			(hide yes)
@@
 		(instances
 			(project "48VERelay"
-				(path "/2d740e7a-a48e-41b8-b74e-ca0ab277f7d9"
-					(reference "U1")
-					(unit 1)
-				)
 				(path "/2d740e7a-a48e-41b8-b74e-ca0ab277f7d9/9acca724-bbf8-479c-b765-a30537109626"
 					(reference "U2")

Commit message: Begin PCB layout
Parts:
- 0685T5000-01: footprint (none) -> Fuse:Fuse_0603_1608Metric
- J10, J11, J12, J13, J14: footprint (none) -> TerminalBlock:TerminalBlock_Xinya_XY308-2.54-3P_1x03_P2.54mm_Horizontal
- R10, R11, R12, R14: value 10k -> 100k
- U2: footprint (none) -> Package_SO:SOIC-18W_7.5x11.6mm_P1.27mm
- renumbered D5 to D4, D4 to D5
Connections:
- removed net COM: 0685T5000-01.2, 0685T5000-2.2, 0685T5000-3.2, 0685T5000-4.2, 0685T5000-5.2, J10.2 (Pin_2), J11.2 (Pin_2), J12.2 (Pin_2), J13.2 (Pin_2), J14.2 (Pin_2)
- removed net NC: J10.3 (Pin_3), J11.3 (Pin_3), J12.3 (Pin_3), J13.3 (Pin_3), J14.3 (Pin_3), K10.12, K11.12, K12.12, K13.12, K14.12
- removed net NO: J10.1 (Pin_1), J11.1 (Pin_1), J12.1 (Pin_1), J13.1 (Pin_1), J14.1 (Pin_1), K10.14, K11.14, K12.14, K13.14, K14.14
- net RELAY_4 renamed MCU_RELAY_4
- removed net RELAY_5: R10.1, R12.1, R13.1, R14.1, U2.1 (I1), U2.2 (I2), U2.3 (I3), U2.5 (I5)
- new net COM_1: 0685T5000-01.2, J10.2 (Pin_2)
- new net COM_2: 0685T5000-2.2, J11.2 (Pin_2)
- new net COM_3: 0685T5000-3.2, J12.2 (Pin_2)
- new net COM_4: 0685T5000-4.2, J13.2 (Pin_2)
- new net COM_5: 0685T5000-5.2, J14.2 (Pin_2)
- new net MCU_RELAY_1: R14.1, U2.1 (I1)
- new net MCU_RELAY_2: R13.1, U2.2 (I2)
- new net MCU_RELAY_3: R12.1, U2.3 (I3)
- new net MCU_RELAY_5: R10.1, U2.5 (I5)
- new net NC_1: J10.3 (Pin_3), K10.12
- new net NC_2: J11.3 (Pin_3), K11.12
- new net NC_3: J12.3 (Pin_3), K12.12
- new net NC_4: J13.3 (Pin_3), K13.12
- new net NC_5: J14.3 (Pin_3), K14.12
- new net NO_1: J10.1 (Pin_1), K10.14
- new net NO_2: J11.1 (Pin_1), K11.14
- new net NO_3: J12.1 (Pin_1), K12.14
- new net NO_4: J13.1 (Pin_1), K13.14
- new net NO_5: J14.1 (Pin_1), K14.14
Changed lines of the file:
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@@
 		)
 	)
-	(label "NO"
+	(label "NO_4"
 		(at 214.63 105.41 0)
 		(effects
@@
 		)
 	)
-	(label "RELAY_5"
+	(label "MCU_RELAY_5"
 		(at 74.93 76.2 0)
 		(effects
@@
 		)
 	)
-	(label "NO"
+	(label "NO_3"
 		(at 214.63 80.01 0)
 		(effects
@@
 		)
 	)
-	(label "NC"
+	(label "NC_5"
 		(at 238.76 142.24 0)
 		(effects
@@
 		)
 	)
-	(label "NO"
+	(label "NO_3"
 		(at 238.76 86.36 0)
 		(effects
@@
 		)
 	)
-	(label "RELAY_4"
+	(label "MCU_RELAY_4"
 		(at 67.31 73.66 0)
 		(effects
@@
 		)
 	)
-	(label "NC"
+	(label "NC_3"
 		(at 209.55 80.01 0)
 		(effects
@@
 		)
 	)
-	(label "NO"
+	(label "NO_1"
 		(at 238.76 35.56 0)
 		(effects
@@
 		)
 	)
-	(label "COM"
+	(label "COM_5"
 		(at 238.76 139.7 0)
 		(effects
@@
 		)
 	)
-	(label "NC"
+	(label "NC_1"
 		(at 238.76 40.64 0)
 		(effects
@@
 		)
 	)
-	(label "NC"
+	(label "NC_2"
 		(at 209.55 54.61 0)
 		(effects
@@
 		)
 	)
-	(label "COM"
+	(label "COM_4"
 		(at 227.33 121.92 0)
 		(effects
@@
 		)
 	)
-	(label "COM"
+	(label "COM_3"
 		(at 227.33 96.52 0)
 		(effects
@@
 		)
 	)
-	(label "RELAY_5"
+	(label "MCU_RELAY_3"
 		(at 59.69 71.12 0)
 		(effects
@@
 		)
 	)
-	(label "NO"
+	(label "NO_4"
 		(at 238.76 111.76 0)
 		(effects
@@
 		)
 	)
-	(label "NC"
+	(label "NC_1"
 		(at 209.55 27.94 0)
 		(effects
@@
 		)
 	)
-	(label "COM"
+	(label "COM_5"
 		(at 227.33 147.32 0)
 		(effects
@@
 		)
 	)
-	(label "RELAY_5"
+	(label "MCU_RELAY_1"
 		(at 44.45 66.04 0)
 		(effects
@@
 		)
 	)
-	(label "NC"
+	(label "NC_2"
 		(at 238.76 66.04 0)
 		(effects
@@
 		)
 	)
-	(label "NO"
+	(label "NO_2"
 		(at 238.76 60.96 0)
 		(effects
@@
 		)
 	)
-	(label "NO"
+	(label "NO_5"
 		(at 238.76 137.16 0)
 		(effects
@@
 		)
 	)
-	(label "COM"
+	(label "COM_2"
 		(at 238.76 63.5 0)
 		(effects
@@
 		)
 	)
-	(label "RELAY_5"
+	(label "MCU_RELAY_2"
 		(at 52.07 68.58 0)
 		(effects
@@
 		)
 	)
-	(label "NC"
+	(label "NC_5"
 		(at 209.55 129.54 0)
 		(effects
@@
 		)
 	)
-	(label "COM"
+	(label "COM_1"
 		(at 227.33 45.72 0)
 		(effects
@@
 		)
 	)
-	(label "COM"
+	(label "COM_2"
 		(at 227.33 71.12 0)
 		(effects
@@
 		)
 	)
-	(label "NC"
+	(label "NC_4"
 		(at 238.76 116.84 0)
 		(effects
@@
 		)
 	)
-	(label "COM"
+	(label "COM_4"
 		(at 238.76 114.3 0)
 		(effects
@@
 		)
 	)
-	(label "NC"
+	(label "NC_4"
 		(at 209.55 105.41 0)
 		(effects
@@
 		)
 	)
-	(label "NO"
+	(label "NO_1"
 		(at 214.63 27.94 0)
 		(effects
@@
 		)
 	)
-	(label "NC"
+	(label "NC_3"
 		(at 238.76 91.44 0)
 		(effects
@@
 		)
 	)
-	(label "NO"
+	(label "NO_5"
 		(at 214.63 129.54 0)
 		(effects
@@
 		)
 	)
-	(label "COM"
+	(label "COM_3"
 		(at 238.76 88.9 0)
 		(effects
@@
 		)
 	)
-	(label "COM"
+	(label "COM_1"
 		(at 238.76 38.1 0)
 		(effects
@@
 		)
 	)
-	(label "NO"
+	(label "NO_2"
 		(at 214.63 54.61 0)
 		(effects
@@
 			)
 		)
-		(property "Footprint" ""
+		(property "Footprint" "TerminalBlock:TerminalBlock_Xinya_XY308-2.54-3P_1x03_P2.54mm_Horizontal"
 			(at 248.92 114.3 0)
 			(hide yes)
@@
 			)
 		)
-		(property "Value" "10k"
+		(property "Value" "100k"
 			(at 78.74 78.994 0)
 			(show_name no)
@@
 		(in_pos_files yes)
 		(dnp no)
-		(property "Reference" "D4"
+		(property "Reference" "D5"
 			(at 113.284 85.598 0)
 			(show_name no)
@@
 			(project "48VERelay"
 				(path "/2d740e7a-a48e-41b8-b74e-ca0ab277f7d9/9acca724-bbf8-479c-b765-a30537109626"
-					(reference "D4")
+					(reference "D5")
 					(unit 1)
 				)
@@
 		(in_pos_files yes)
 		(dnp no)
-		(property "Reference" "D5"
+		(property "Reference" "D4"
 			(at 127.254 83.058 0)
 			(show_name no)
@@
 			(project "48VERelay"
 				(path "/2d740e7a-a48e-41b8-b74e-ca0ab277f7d9/9acca724-bbf8-479c-b765-a30537109626"
-					(reference "D5")
+					(reference "D4")
 					(unit 1)
 				)
@@
 			)
 		)
-		(property "Value" "10k"
+		(property "Value" "100k"
 			(at 71.12 76.962 0)
 			(show_name no)
@@
 			)
 		)
-		(property "Footprint" ""
+		(property "Footprint" "TerminalBlock:TerminalBlock_Xinya_XY308-2.54-3P_1x03_P2.54mm_Horizontal"
 			(at 248.92 88.9 0)
 			(hide yes)
@@
 			)
 		)
-		(property "Footprint" ""
+		(property "Footprint" "Fuse:Fuse_0603_1608Metric"
 			(at 222.25 45.72 0)
 			(hide yes)
@@
 			)
 		)
-		(property "Value" "10k"
+		(property "Value" "100k"
 			(at 48.768 69.088 0)
 			(show_name no)
@@
 			)
 		)
-		(property "Value" "10k"
+		(property "Value" "100k"
 			(at 63.5 73.66 0)
 			(show_name no)
@@
 			)
 		)
-		(property "Footprint" ""
+		(property "Footprint" "TerminalBlock:TerminalBlock_Xinya_XY308-2.54-3P_1x03_P2.54mm_Horizontal"
 			(at 248.92 139.7 0)
 			(hide yes)
@@
 			)
 		)
-		(property "Footprint" ""
+		(property "Footprint" "TerminalBlock:TerminalBlock_Xinya_XY308-2.54-3P_1x03_P2.54mm_Horizontal"
 			(at 248.92 38.1 0)
 			(hide yes)
@@
 			)
 		)
-		(property "Footprint" ""
+		(property "Footprint" "Package_SO:SOIC-18W_7.5x11.6mm_P1.27mm"
 			(at 96.52 87.63 0)
 			(hide yes)
@@
 			)
 		)
-		(property "Footprint" ""
+		(property "Footprint" "TerminalBlock:TerminalBlock_Xinya_XY308-2.54-3P_1x03_P2.54mm_Horizontal"
 			(at 248.92 63.5 0)
 			(hide yes)
