File: RelatBoard/48VRelay/48VERelay/Outputs.kicad_sch (KiCad schematic)
At the start: 31 parts, among them J10 Screw_Terminal_01x03, J11 Screw_Terminal_01x03, J12 Screw_Terminal_01x03, J13 Screw_Terminal_01x03, J14 Screw_Terminal_01x03, K10 G2RL-1-E, K11 G2RL-1-E, K12 G2RL-1-E, K13 G2RL-1-E, K14 G2RL-1-E, U2 ULN2803A

Commit message: Fixed jtag, fixed diff pair routing, removed fuses
Parts:
- removed F1, F2, F5: 0685T5000, Fuse:Fuse_1206_3216Metric, symbol Device:Fuse_Small
- removed F3, F4: 0685T5000-01, Fuse:Fuse_1206_3216Metric, symbol Device:Fuse_Small
Connections:
- net COM_1: now also K10.11
- net COM_2: now also K11.11
- net COM_3: now also K12.11
- net COM_4: now also K13.11
- net COM_5: now also K14.11
