File: RelatBoard/48VRelay/48VERelay/48VERelay.kicad_pcb (KiCad board)
At the start: 2 copper layers, 9 parts, among them J2 RJ45_Hanrun_HR911105A_Horizon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, K10 G2RL-1-E, K11 G2RL-1-E, K12 G2RL-1-E, K13 G2RL-1-E, K14 G2RL-1-E, U1 ESP32-WROOM-32UE, U3 W5500

Commit message: Begin PCB layout
Parts:
- added 0685T5000-01: Fuse_Small, Fuse:Fuse_0603_1608Metric, F.Cu at (268.5, 58.0)
- added 0685T5000-2: Fuse_Small, Fuse:Fuse_0603_1608Metric, F.Cu at (268.5, 72.0)
- added 0685T5000-3: Fuse_Small, Fuse:Fuse_0603_1608Metric, F.Cu at (268.0, 85.5)
- added 0685T5000-4: Fuse_Small, Fuse:Fuse_0603_1608Metric, F.Cu at (268.0, 99.5)
- added 0685T5000-5: Fuse_Small, Fuse:Fuse_0603_1608Metric, F.Cu at (268.0, 113.5)
- added C1: 10uF, Capacitor_SMD:C_0805_2012Metric, F.Cu at (148.9, 116.2)
- added C10: 100nF - Ceramic, Capacitor_SMD:C_0201_0603Metric, F.Cu at (70.5, 140.5)
- added C11: 0.1uF, Capacitor_SMD:C_0201_0603Metric, F.Cu at (152.4, 132.6)
- added C12: 0.1uF, Capacitor_SMD:C_0201_0603Metric, F.Cu at (152.4, 134.4)
- added C13: 0.1uF, Capacitor_SMD:C_0201_0603Metric, F.Cu at (154.8, 125.6)
- added C14: 0.1uF, Capacitor_SMD:C_0201_0603Metric, F.Cu at (154.8, 127.4)
- added C15: 0.1uF, Capacitor_SMD:C_0201_0603Metric, F.Cu at (154.8, 129.1)
- added C16: 0.1uF, Capacitor_SMD:C_0201_0603Metric, F.Cu at (154.8, 130.9)
- added C17: 6.8nF, Capacitor_SMD:C_0201_0603Metric, F.Cu at (154.8, 132.6)
- added C18: 10uF / 16V, Capacitor_SMD:C_0805_2012Metric, F.Cu at (148.9, 128.3)
- added C19: 6.8nF, Capacitor_SMD:C_0201_0603Metric, F.Cu at (154.8, 134.4)
- added C2: 10uF, Capacitor_SMD:C_0805_2012Metric, F.Cu at (148.9, 119.2)
- added C20: 10nF, Capacitor_SMD:C_0201_0603Metric, F.Cu at (188.4, 136.6)
- added C21: 18pF, Capacitor_SMD:C_0201_0603Metric, F.Cu at (157.3, 125.6)
- added C22: 18pF, Capacitor_SMD:C_0201_0603Metric, F.Cu at (157.3, 127.4)
- added C23: 10nF, Capacitor_SMD:C_0201_0603Metric, F.Cu at (157.3, 129.1)
- added C24: 1uF - Ceramic, Capacitor_SMD:C_0805_2012Metric, F.Cu at (75.5, 97.0)
- added C25: 100nF, Capacitor_SMD:C_0201_0603Metric, F.Cu at (71.5, 140.5)
- added C26: 10uF, Capacitor_SMD:C_0805_2012Metric, F.Cu at (68.0, 140.5)
- added C27: 10uF, Capacitor_SMD:C_0805_2012Metric, F.Cu at (151.9, 152.2)
- added C28: 10uF, Capacitor_SMD:C_0603_1608Metric, F.Cu at (151.9, 155.3)
- added C29: 10uF, Capacitor_SMD:C_0603_1608Metric, F.Cu at (151.9, 158.3)
- added C3: 0.1uF, Capacitor_SMD:C_0201_0603Metric, F.Cu at (152.4, 125.6)
- added C30: 22uF, Capacitor_SMD:C_0805_2012Metric, F.Cu at (156.9, 155.2)
- added C31: 22uF, Capacitor_SMD:C_0805_2012Metric, F.Cu at (156.9, 158.5)
- added C32: 1uF, Capacitor_SMD:C_0201_0603Metric, F.Cu at (155.3, 150.8)
- added C33: 1uF, Capacitor_SMD:C_0201_0603Metric, F.Cu at (155.3, 152.6)
- added C34: 1uF, Capacitor_SMD:C_0805_2012Metric, F.Cu at (151.9, 161.3)
- added C35: 1uF, Capacitor_SMD:C_0805_2012Metric, F.Cu at (151.9, 164.3)
- added C4: 0.1uF, Capacitor_SMD:C_0201_0603Metric, F.Cu at (152.4, 127.4)
- added C5: 4.7uF - Eth Reference Cap, Capacitor_SMD:C_0805_2012Metric, F.Cu at (148.9, 122.2)
- added C6: 22nF, Capacitor_SMD:C_0201_0603Metric, F.Cu at (152.4, 129.1)
- added C7: 0.1uF, Capacitor_SMD:C_0201_0603Metric, F.Cu at (152.4, 130.9)
- added C8: 10uF, Capacitor_SMD:C_0805_2012Metric, F.Cu at (148.9, 125.2)
- added C9: C_Small, Capacitor_SMD:C_0201_0603Metric, F.Cu at (69.5, 140.5)
- added D1: LED VO-PT2012SEAC, LED_SMD:LED_0201_0603Metric, F.Cu at (184.3, 141.6)
- added D2: LED VO-PT2012SEAC, LED_SMD:LED_0201_0603Metric, F.Cu at (184.3, 143.3)
- added D3: LED VO-PT2012SEAC, LED_SMD:LED_0201_0603Metric, F.Cu at (225.0, 90.0)
- added D4: LED VO-PT2012SEAC, LED_SMD:LED_0201_0603Metric, F.Cu at (229.0, 101.5)
- added D5: LED VO-PT2012SEAC, LED_SMD:LED_0201_0603Metric, F.Cu at (230.0, 119.0)
- added D6: LED, LED_SMD:LED_0201_0603Metric, F.Cu at (160.0, 128.6)
- added J1: 12, Connector_BarrelJack:BarrelJack_CUI_PJ-102AH_Horizontal, F.Cu at (55.5, 141.0)
- added J10: Screw_Terminal_01x03, TerminalBlock:TerminalBlock_Xinya_XY308-2.54-3P_1x03_P2.54mm_Horizontal, F.Cu at (276.5, 62.5)
- added J11: Screw_Terminal_01x03, TerminalBlock:TerminalBlock_Xinya_XY308-2.54-3P_1x03_P2.54mm_Horizontal, F.Cu at (276.3, 75.5)
- added J12: Screw_Terminal_01x03, TerminalBlock:TerminalBlock_Xinya_XY308-2.54-3P_1x03_P2.54mm_Horizontal, F.Cu at (276.5, 89.5)
- added J13: Screw_Terminal_01x03, TerminalBlock:TerminalBlock_Xinya_XY308-2.54-3P_1x03_P2.54mm_Horizontal, F.Cu at (276.5, 102.5)
- added J14: Screw_Terminal_01x03, TerminalBlock:TerminalBlock_Xinya_XY308-2.54-3P_1x03_P2.54mm_Horizontal, F.Cu at (276.5, 116.5)
- added L1: MH1608-121Y, Library:IND_BOURNS_MH1608, F.Cu at (107.3, 155.0)
- added L2: 1.5uH, Library:IND_XFL4020_COC-M, F.Cu at (93.0, 94.5)
- added L3: XFL4020-152MEC, Library:IND_XFL4020_COC-M, F.Cu at (118.2, 147.7)
- added R1: 2.2k, Resistor_SMD:R_0603_1608Metric, F.Cu at (232.2, 61.5)
- added R10: 10k, Resistor_SMD:R_0603_1608Metric, F.Cu at (204.0, 83.5)
- added R11: 10k, Resistor_SMD:R_0603_1608Metric, F.Cu at (204.0, 81.5)
- added R12: 10k, Resistor_SMD:R_0603_1608Metric, F.Cu at (180.8, 144.5)
- added R13: 10k, Resistor_SMD:R_0603_1608Metric, F.Cu at (180.8, 147.0)
- added R14: 10k, Resistor_SMD:R_0603_1608Metric, F.Cu at (180.8, 149.5)
- added R15: 330, Resistor_SMD:R_0603_1608Metric, F.Cu at (83.5, 51.5)
- added R16: 33, Resistor_SMD:R_0603_1608Metric, F.Cu at (153.2, 123.5)
- added R17: 33, Resistor_SMD:R_0603_1608Metric, F.Cu at (157.2, 116.0)
- added R18: 49.9 1%, Resistor_SMD:R_0603_1608Metric, F.Cu at (157.2, 118.5)
- added R19: 49.9 1%, Resistor_SMD:R_0805_2012Metric, F.Cu at (160.7, 126.2)
- added R2: 2.2k, Resistor_SMD:R_0603_1608Metric, F.Cu at (192.0, 93.5)
- added R20: 10 1%, Resistor_SMD:R_0603_1608Metric, F.Cu at (157.2, 121.0)
- added R21: 49.9 1%, Resistor_SMD:R_0603_1608Metric, F.Cu at (157.2, 123.5)
- added R22: 49.9 1%, Resistor_SMD:R_0603_1608Metric, F.Cu at (161.2, 116.0)
- added R23: 0, Resistor_SMD:R_0603_1608Metric, F.Cu at (161.2, 118.5)
- added R24: 1M, Resistor_SMD:R_0603_1608Metric, F.Cu at (161.2, 121.0)
- added R25: 10k, Resistor_SMD:R_0603_1608Metric, F.Cu at (129.5, 116.5)
- added R26: 680kΩ, Resistor_SMD:R_0603_1608Metric, F.Cu at (129.5, 119.0)
- added R27: 130kΩ, Resistor_SMD:R_0603_1608Metric, F.Cu at (129.5, 121.5)
- added R28: 100kΩ, Resistor_SMD:R_0603_1608Metric, F.Cu at (129.5, 124.0)
- added R29: 330, Resistor_SMD:R_0603_1608Metric, F.Cu at (161.2, 123.5)
- added R3: 2.2k, Resistor_SMD:R_0603_1608Metric, F.Cu at (176.8, 144.5)
- added R4: 2.2k, Resistor_SMD:R_0603_1608Metric, F.Cu at (176.8, 147.0)
- added R5: 2.2k, Resistor_SMD:R_0603_1608Metric, F.Cu at (232.0, 101.5)
- added R6: 12.4k 1% - Ethernet external reference, Resistor_SMD:R_0603_1608Metric, F.Cu at (153.2, 116.0)
- added R7: 33, Resistor_SMD:R_0603_1608Metric, F.Cu at (153.2, 118.5)
- added R8: 33, Resistor_SMD:R_0603_1608Metric, F.Cu at (153.2, 121.0)
- added R9: 330, Resistor_SMD:R_0603_1608Metric, F.Cu at (77.7, 51.5)
- added U2: ULN2803A, Package_SO:SOIC-18W_7.5x11.6mm_P1.27mm, F.Cu at (215.0, 83.0)
- added U4: 3A 32V, Fuse:Fuse_1206_3216Metric, F.Cu at (63.0, 138.0)
- added U5: TPS630701RNMR, Library:RNM0015A, F.Cu at (78.5, 138.5)
- added U6: TLV1117LV33DCYR, Library:DCY0004A_M, F.Cu at (110.0, 84.5)
- added U7: TVS1800DRVR, Library:DRV0006A_NV, F.Cu at (71.2, 113.3)
- added U8: TLV1117LV33DCYR, Library:DCY0004A_M, F.Cu at (129.5, 85.0)
- added Y2: ABM3C-25.000MHZ-D4Y-T, Library:CRYSTAL_ABM3C_ABR-M, F.Cu at (110.1, 134.7)
- moved U3 38.3 mm to (87.8, 71.2)
- moved J2 30.9 mm to (62.1, 58.1)
- moved K10 15.0 mm to (237.5, 68.7)
- moved K11 11.5 mm to (237.5, 82.2)
- moved TVS1 11.4 mm to (141.0, 97.9)
- moved K12 7.50 mm to (237.5, 95.7)
- moved K13 3.50 mm to (237.5, 109.2)
Connections:
- net /MCU/RELAY_1 renamed /MCU/MCU_RELAY_1
- net /MCU/RELAY_2 renamed /MCU/MCU_RELAY_2
- net /MCU/RELAY_3 renamed /MCU/MCU_RELAY_3
- net /MCU/RELAY_4 renamed /MCU/MCU_RELAY_4
- net /MCU/RELAY_5 renamed /MCU/MCU_RELAY_5
- K10 pad 12: /Outputs/NC -> /Outputs/NC_1
- K10 pad 14: /Outputs/NO -> /Outputs/NO_1
- K11 pad 12: /Outputs/NC -> /Outputs/NC_2
- K11 pad 14: /Outputs/NO -> /Outputs/NO_2
- K12 pad 12: /Outputs/NC -> /Outputs/NC_3
- K12 pad 14: /Outputs/NO -> /Outputs/NO_3
- K13 pad 12: /Outputs/NC -> /Outputs/NC_4
- K13 pad 14: /Outputs/NO -> /Outputs/NO_4
- K14 pad 12: /Outputs/NC -> /Outputs/NC_5
- K14 pad 14: /Outputs/NO -> /Outputs/NO_5

Commit message: 5v5 Buck Added
Parts:
- removed L2: 1.5uH, Library:IND_XFL4020_COC-M
- removed R26: 680kΩ, Resistor_SMD:R_0603_1608Metric
- removed R27: 130kΩ, Resistor_SMD:R_0603_1608Metric
- removed TVS1: SMBJ18A, Package_SON:WSON-6-1EP_2x2mm_P0.65mm_EP1x1.6mm
- added J3: Conn_ARM_SWD_TagConnect_TC2030-NL, Connector:Tag-Connect_TC2030-IDC-NL_2x03_P1.27mm_Vertical, F.Cu at (64.0, 166.3)
- R10, R11, R12, R14: value 10k -> 100k
- moved D6 103.6 mm to (56.9, 118.4)
- moved R29 100.9 mm to (60.4, 119.4)
- moved C6 100.1 mm to (75.5, 65.0), turned to 180 degrees
- moved C11 95.0 mm to (78.8, 72.5)
- moved C12 93.5 mm to (79.3, 76.0)
- moved C35 92.4 mm to (88.0, 97.5), turned to 180 degrees
- moved C32 91.9 mm to (90.2, 86.0), turned to 180 degrees
- moved C13 91.1 mm to (82.3, 70.5)
- moved C34 90.2 mm to (104.5, 84.5), turned to 90 degrees
- moved D1 88.7 mm to (229.0, 65.0)
- moved C15 86.4 mm to (84.8, 78.5)
- moved C14 83.5 mm to (89.8, 75.0)
- moved C18 82.5 mm to (90.0, 70.5)
- moved C16 82.2 mm to (90.3, 80.0)
- moved C5 80.5 mm to (84.5, 74.0)
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Connections:
- net Net-(J1-Pad1) renamed /Power/VIN_12V
- U5 pad 5: Net-(U5-FB) -> +5V
Routing:
- net +12V: track 0.00 -> 24.4 mm
- net /Power/VIN_12V: track 0.00 -> 19.2 mm
- net +5V: track 0.00 -> 12.3 mm
- net Net-(U5-L1): track 0.00 -> 7.09 mm
- net Net-(U5-PG): track 0.00 -> 6.20 mm
- net Net-(U5-L2): track 0.00 -> 6.07 mm
- net Net-(C26-Pad2): track 0.00 -> 4.83 mm
- net Net-(U5-EN): track 0.00 -> 2.41 mm
- net GND: track 0.00 -> 1.70 mm, vias 0 -> 1
- net Net-(U5-VAUX): track 0.00 -> 1.64 mm
- net (no net): vias 0 -> 1

Commit message: Fix 12V->5V add power plane
Parts:
- moved 0685T5000-2 106.1 mm to (167.0, 103.0)
- moved C20 105.0 mm to (101.7, 74.0)
- moved J11 104.2 mm to (175.3, 101.0)
- moved 0685T5000-01 104.2 mm to (167.5, 83.5)
- moved 0685T5000-3 104.2 mm to (167.0, 111.0)
- moved 0685T5000-4 104.2 mm to (167.0, 125.0)
- moved 0685T5000-5 104.2 mm to (167.0, 139.0)
- moved D1 104.2 mm to (128.0, 90.5)
- moved D2 104.2 mm to (128.0, 104.0)
- moved D3 104.2 mm to (128.0, 117.5)
- moved D4 104.2 mm to (128.0, 131.0)
- moved D5 104.2 mm to (128.0, 145.0)
- moved J10 104.2 mm to (175.5, 88.0)
- moved J12 104.2 mm to (175.5, 115.0)
- moved J13 104.2 mm to (175.5, 128.0)
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Connections:
- C26 pad 2: Net-(C26-Pad2) -> GND
- C27 pad 2: Net-(C26-Pad2) -> GND
- R25 pad 1: Net-(C26-Pad2) -> +12V
Routing:
- net /Power/VIN_12V: track 19.2 -> 9.41 mm
- net Net-(C26-Pad2): track 4.83 -> 0.00 mm
- net Net-(U5-EN): track 2.41 -> 5.61 mm
- net +12V: track 24.4 -> 21.3 mm
- net GND: track 1.70 -> 2.64 mm, vias 1 -> 2
- net (no net): vias 1 -> 0
- added copper zone on F.Cu, net +12V
- added copper zone on B.Cu, net GND
