File: RelatBoard/48VRelay/48VERelay/48VERelay.kicad_pcb (KiCad board)
At the start: 2 copper layers, 97 parts, among them J1 12, J10 Screw_Terminal_01x03, J11 Screw_Terminal_01x03, J12 Screw_Terminal_01x03, J13 Screw_Terminal_01x03, J14 Screw_Terminal_01x03, J2 RJ45_Hanrun_HR911105A_Horizon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, J3 Conn_ARM_SWD_TagConnect_TC203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, K10 G2RL-1-E, K11 G2RL-1-E, K12 G2RL-1-E, K13 G2RL-1-E, K14 G2RL-1-E, U1 ESP32-WROOM-32UE, U2 ULN2803A, U3 W5500, U4 3A 32V, U5 TPS630701RNMR, U6 TLV1117LV33DCYR, U7 TVS1800DRVR, U8 TLV1117LV33DCYR, Y2 ABM3C-25.000MHZ-D4Y-T

Commit message: update layout
Parts:
- removed U6, U8: TLV1117LV33DCYR, Library:DCY0004A_M
- added 12V: TestPoint_Pad_D1.5mm, TestPoint:TestPoint_Pad_D1.5mm, F.Cu at (65.5, 52.8)
- added GND: , , F.Cu at (59.2, 55.5)
- added U10: TLV1117LV33DCYR, Library:TLV1117-33IDCYR, F.Cu at (51.0, 63.0)
- added U9: TLV1117LV33DCYR, Library:TLV1117-33IDCYR, F.Cu at (66.0, 75.0)
- C9: value C_Small -> 100uF - Electrolytic; footprint Capacitor_SMD:C_0201_0603Metric -> Capacitor_SMD:C_Elec_6.3x7.7
- moved R19 57.9 mm to (43.4, 84.5)
- moved R17 53.9 mm to (46.5, 84.5)
- moved R8 51.3 mm to (44.3, 86.8)
- moved R6 47.2 mm to (49.6, 84.2)
- moved 0685T5000-01 47.0 mm to (154.7, 38.3)
- moved 0685T5000-2 47.0 mm to (154.2, 57.8)
- moved 0685T5000-3 47.0 mm to (154.2, 65.8)
- moved 0685T5000-4 47.0 mm to (154.2, 79.8)
- moved 0685T5000-5 47.0 mm to (154.2, 93.8)
- moved D1 47.0 mm to (115.2, 45.3)
- moved D2 47.0 mm to (115.2, 58.8)
- moved D3 47.0 mm to (115.2, 72.3)
- moved D4 47.0 mm to (115.2, 85.8)
- moved D5 47.0 mm to (115.2, 99.8)
- moved J10 47.0 mm to (162.7, 42.7)
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Routing:
- net +3V3 MCU: track 0.00 -> 15.1 mm
- net +5V: track 12.3 -> 19.6 mm, vias 0 -> 2
- net Net-(U5-EN): track 5.61 -> 9.40 mm
- net GND: track 2.64 -> 5.81 mm, vias 2 -> 30
- net /MCU/JTAG_RESET: track 0.00 -> 3.04 mm
- net Net-(U5-L1): track 7.09 -> 8.15 mm
- net Net-(U5-PG): track 6.20 -> 7.20 mm
- net Net-(U5-L2): track 6.07 -> 7.03 mm
- net Net-(U5-VAUX): track 1.64 -> 1.07 mm
- added copper zone on F.Cu, net +3V3 MCU
- added copper zone on F.Cu, net +5V
- added copper zone on F.Cu, net GND
