File: RelatBoard/48VRelay/48VERelay/48VERelay.kicad_pcb (KiCad board)
At the start: 4 copper layers, 117 x 92 mm, 116 parts, among them J1 12, J10 Screw_Terminal_01x03, J11 Screw_Terminal_01x03, J12 Screw_Terminal_01x03, J13 Screw_Terminal_01x03, J14 Screw_Terminal_01x03, J2 RJ45_Hanrun_HR911105A_Horizon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, J3 B4B-PH-SM4-TB, J5 TC2030, K10 G2RL-1-E, K11 G2RL-1-E, K12 G2RL-1-E, K13 G2RL-1-E, K14 G2RL-1-E, SW5 ENABLE, SW6 RESET, U1 ESP32-WROOM-32UE, U10 TLV1117LV33DCYR, U2 ULN2803A, U3 W5500, U4 3A 32V, U5 TPS630701RNMR, U7 TVS1800DRVR, U9 TLV1117LV33DCYR, Y2 ABM3C-25.000MHZ-D4Y-T

Commit message: Final design
Parts:
- removed F1, F2, F5: 0685T5000, Fuse:Fuse_1206_3216Metric
- removed F3, F4: 0685T5000-01, Fuse:Fuse_1206_3216Metric
- removed the G*** at (85.0, 38.5)
- removed J5: TC2030, Connector:Tag-Connect_TC2030-IDC-NL_2x03_P1.27mm_Vertical
- removed K10, K11, K12, K13, K14: G2RL-1-E, Relay_THT:Relay_SPDT_Omron_G2RL-1-E
- added J4: TC2050, Connector:Tag-Connect_TC2050-IDC-NL_2x05_P1.27mm_Vertical, F.Cu at (79.2, 105.7)
- added K1: G2R-1-E DC12, Relay_THT:RELAY_G2R-1-E AC12_OMR, F.Cu at (117.8, 46.6)
- added K2: G2R-1-E DC12, Relay_THT:RELAY_G2R-1-E AC12_OMR, F.Cu at (117.4, 63.0)
- added K3: G2R-1-E DC12, Relay_THT:RELAY_G2R-1-E AC12_OMR, F.Cu at (117.4, 80.0)
- added K4: G2R-1-E DC12, Relay_THT:RELAY_G2R-1-E AC12_OMR, F.Cu at (117.4, 97.2)
- added K5: G2R-1-E DC12, Relay_THT:RELAY_G2R-1-E AC12_OMR, F.Cu at (117.5, 114.2)
- 3V3 Eth: moved to F.Cu
- 3V3A: moved to F.Cu
- Y2: footprint Library:CRYSTAL_ABM3C_ABR-M -> Crystal:Crystal_SMD_Abracon_ABM3C-4Pin_5.0x3.2mm
- moved R16 24.9 mm to (52.8, 96.8), turned to 0 degrees
- moved R6 24.5 mm to (51.7, 94.5), turned to 180 degrees
- moved R17 23.1 mm to (52.8, 95.2), turned to 0 degrees
- moved C12 20.5 mm to (48.5, 92.0), turned to 90 degrees
- moved R20 20.3 mm to (46.2, 106.0), turned to -90 degrees
- moved C6 19.8 mm to (46.2, 107.9)
- moved C13 19.4 mm to (53.2, 92.0), turned to 90 degrees
- moved C15 19.4 mm to (50.5, 92.0), turned to 90 degrees
- moved R21 17.2 mm to (55.0, 97.2), turned to -90 degrees
- moved C21 17.2 mm to (47.8, 75.2), turned to 90 degrees
- moved R22 15.3 mm to (55.0, 95.0), turned to 90 degrees
- moved C16 14.6 mm to (54.0, 89.5), turned to 180 degrees
- moved R23 14.2 mm to (47.0, 77.5), turned to 90 degrees
- moved C17 14.1 mm to (56.2, 96.8), turned to 0 degrees
- moved C14 12.7 mm to (54.0, 88.5), turned to 180 degrees
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Routing:
- net /MCU/Ether_RESET: track 42.9 -> 83.3 mm
- net /MCU/Ether_INT: track 17.2 -> 55.0 mm, vias 0 -> 2
- net /MCU/Ether_MOSI: track 18.8 -> 55.0 mm, vias 0 -> 2
- net /MCU/Ether_MISO: track 19.9 -> 54.3 mm, vias 0 -> 2
- net /MCU/Ether_SCLK: track 21.0 -> 54.0 mm, vias 0 -> 2
- net RX_CT: track 53.4 -> 21.9 mm
- net /MCU/Ether_CS: track 20.2 -> 51.2 mm
- net GND: track 101.1 -> 132.0 mm, vias 71 -> 176
- net /MCU/PHY_R_TXN: track 32.1 -> 3.26 mm
- net /MCU/PHY_R_TXP: track 30.6 -> 2.87 mm
- net RX_N: track 42.2 -> 19.2 mm, vias 2 -> 0
- net RX_P: track 40.5 -> 19.1 mm
- net +3V3 Eth: track 73.7 -> 93.9 mm, vias 4 -> 5
- net Net-(F3-Pad1): track 16.5 -> 0.00 mm
- net Net-(F2-Pad1): track 16.3 -> 0.00 mm
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Other:
- board size 117 x 92 mm -> 110 x 92 mm
- board text added: "220V AC 16A MAX"
- board text added: "3v3 ONLY"
- board text added: "5 Channel Relay"
- board text added: "52V DC 2.5A MAX"
- board text added: "QL5CHBSCRLY"
- board text added: "Qilon"

Commit message: update schematic
Routing:
- net +3V3A: track 81.4 -> 80.0 mm, vias 9 -> 8

Commit message: revA update
Routing:
- net +12V: track 208.2 -> 203.7 mm
- net /Outputs/Relay_2: track 10.7 -> 14.5 mm
Changed lines of the file:
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@@
 	)
 	(segment
-		(start 103.9375 59.25)
-		(end 101.6875 61.5)
-		(width 1.016)
-		(layer "F.Cu")
-		(net "+12V")
-	)
-	(segment
-		(start 105.25 59.25)
-		(end 103.9375 59.25)
-		(width 1.016)
-		(layer "F.Cu")
-		(net "+12V")
-	)
-	(segment
 		(start 70 45.876993)
 		(end 69.8968 45.980193)
@@
 	)
 	(segment
+		(start 105.1646 59.1646)
+		(end 105.25 59.25)
+		(width 0.9144)
+		(layer "F.Cu")
+		(net "/Outputs/Relay_2")
+	)
+	(segment
 		(start 101.4388 58.0388)
 		(end 101.4388 59.1646)
 		(width 0.9144)
 		(layer "F.Cu")
+		(net "/Outputs/Relay_2")
+	)
+	(segment
+		(start 101.4388 59.1646)
+		(end 105.1646 59.1646)
+		(width 0.9144)
+		(layer "F.Cu")
