File: RelatBoard/48VRelay/48VERelay/Power.kicad_sch (KiCad schematic)
At the start: 23 parts, among them J1 12, U4 3A 32V, U5 TPS630701RNMR, U6 TLV1117LV33DCYR, U7 TVS1800DRVR, U8 TLV1117LV33DCYR

Commit message: update layout
Parts:
- removed U6, U8: TLV1117LV33DCYR, Library:DCY0004A_M, symbol 2026-06-15_04-40-12:TLV1117LV33DCYR
- added U10, U9: TLV1117LV33DCYR, Library:TLV1117-33IDCYR, symbol 2026-06-15_04-40-12:TLV1117LV33DCYR
- C9: value C_Small -> 100uF - Electrolytic; footprint Capacitor_SMD:C_0201_0603Metric -> Capacitor_SMD:C_Elec_6.3x7.7
Connections:
- net +3V3 Eth: now also U10.2 (OUT), U10.4 (TAB)
- net +3V3 MCU: now also U9.2 (OUT), U9.4 (TAB)
- net +5V: now also U10.3 (IN), U9.3 (IN)
- net GND: now also U10.1 (GND), U9.1 (GND)
