File: RelatBoard/48VRelay/48VERelay/Power.kicad_sch (KiCad schematic)
At the start: 23 parts, among them J1 12, U10 TLV1117LV33DCYR, U4 3A 32V, U5 TPS630701RNMR, U7 TVS1800DRVR, U9 TLV1117LV33DCYR

Commit message: update txrx routing length
Changed lines of the file:
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@@
-		)
-	)
-	(label "ETH_PWR"
-		(at 125.73 168.91 0)
-		(effects
-			(font
-				(size 1.27 1.27)
-			)
-			(justify left bottom)
-		)
-	)
-	(label "MCU_PWR"
-		(at 125.73 144.78 0)
-		(effects
-			(font
-				(size 1.27 1.27)
-			)
-			(justify left bottom)
 		)
 	)
