File: RelatBoard/48VRelay/48VERelay/_restore_backup_2026-07-11T22-01-59-558/MCU.kicad_sch (KiCad schematic)
At the start: 40 parts, among them U1 ESP32-WROOM-32UE, U3 W5500, Y2 ABM3C-25.000MHZ-D4Y-T

Commit message: Route ethernet
Parts:
- removed R26: 10kΩ, symbol Device:R
- added J3: Conn_ARM_SWD_TagConnect_TC2030-NL, Connector:Tag-Connect_TC2030-IDC-NL_2x03_P1.27mm_Vertical, symbol Connector:Conn_ARM_SWD_TagConnect_TC2030-NL
- R19: footprint Resistor_SMD:R_0201_0603Metric -> Capacitor_SMD:C_0201_0603Metric
- R21, R22: footprint Resistor_SMD:R_0201_0603Metric -> Resistor_SMD:R_0603_1608Metric
Connections:
- net ACT_LED renamed ACT LED
- net LINK_LED renamed LINK LED
Changed lines of the file:
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@@
 	)
 	(junction
-		(at 62.23 50.8)
-		(diameter 0)
-		(color 0 0 0 0)
-	)
-	(junction
 		(at 210.82 76.2)
 		(diameter 0)
@@
 	(wire
 		(pts
-			(xy 62.23 40.64) (xy 62.23 43.18)
-		)
-		(stroke
-			(width 0)
-			(type default)
-		)
-	)
-	(wire
-		(pts
 			(xy 115.57 78.74) (xy 109.22 78.74)
 		)
@@
 	(wire
 		(pts
-			(xy 59.69 50.8) (xy 62.23 50.8)
-		)
-		(stroke
-			(width 0)
-			(type default)
-		)
-	)
-	(wire
-		(pts
 			(xy 85.09 41.91) (xy 90.17 41.91)
 		)
@@
 	(wire
 		(pts
-			(xy 62.23 50.8) (xy 78.74 50.8)
+			(xy 64.77 50.8) (xy 78.74 50.8)
 		)
 		(stroke
@@
 		)
 	)
-	(label "LINK_LED"
+	(label "LINK LED"
 		(at 212.09 129.54 0)
 		(effects
@@
 		)
 	)
-	(label "MCU_PWR"
-		(at 62.23 43.18 180)
-		(effects
-			(font
-				(size 1.27 1.27)
-			)
-			(justify right bottom)
-		)
-	)
 	(label "JTAG_VTREF"
 		(at 97.79 36.83 0)
@@
 		)
 	)
-	(label "ACT_LED"
+	(label "ACT LED"
 		(at 212.09 134.62 0)
 		(effects
@@
 	)
 	(label "JTAG_RESET"
-		(at 59.69 50.8 180)
+		(at 64.77 50.8 0)
 		(effects
 			(font
 				(size 1.27 1.27)
 			)
-			(justify right bottom)
+			(justify left bottom)
 		)
 	)
@@
 			)
 		)
-		(property "Footprint" "Resistor_SMD:R_0201_0603Metric"
+		(property "Footprint" "Resistor_SMD:R_0603_1608Metric"
 			(at 234.95 111.76 0)
 			(hide yes)
@@
 			)
 		)
-		(property "Footprint" "Resistor_SMD:R_0201_0603Metric"
+		(property "Footprint" "Resistor_SMD:R_0603_1608Metric"
 			(at 228.6 110.49 0)
 			(hide yes)
@@
 	)
 	(symbol
-		(lib_id "Device:R")
-		(at 62.23 46.99 0)
+		(lib_id "Device:C_Small")
+		(at 219.71 149.86 0)
 		(unit 1)
 		(body_style 1)
@@
 		(in_pos_files yes)
 		(dnp no)
-		(property "Reference" "R26"
-			(at 66.802 46.99 90)
+		(fields_autoplaced yes)
+		(property "Reference" "C5"
+			(at 222.25 148.5962 0)
 			(show_name no)
 			(do_not_autoplace no)
@@
 					(size 1.27 1.27)
 				)
+				(justify left)
 			)
 		)
-		(property "Value" "10kΩ"
-			(at 64.77 46.99 90)
+		(property "Value" "4.7uF - Eth Reference Cap"
+			(at 222.25 151.1363 0)
 			(show_name no)
 			(do_not_autoplace no)
 			(effects
 				(font
-					(size 1.27 1.27)
+					(size 0.8128 0.8128)
 				)
+				(justify left)
 			)
 		)
-		(property "Footprint" ""
-			(at 60.452 46.99 90)
+		(property "Footprint" "Capacitor_SMD:C_0201_0603Metric"
+			(at 219.71 149.86 0)
 			(hide yes)
 			(show_name no)
@@
 		)
 		(property "Datasheet" ""
-			(at 62.23 46.99 0)
+			(at 219.71 149.86 0)
 			(hide yes)
 			(show_name no)
@@
 			)
 		)
-		(property "Description" "Resistor"
-			(at 62.23 46.99 0)
+		(property "Description" "Unpolarized capacitor, small symbol"
+			(at 219.71 149.86 0)
 			(hide yes)
 			(show_name no)
@@
 			(project "48VERelay"
 				(path "/2d740e7a-a48e-41b8-b74e-ca0ab277f7d9/856446f6-474b-446a-aa46-e1d1fc2a9600"
-					(reference "R26")
+					(reference "C5")
 					(unit 1)
 				)
@@
 	)
 	(symbol
-		(lib_id "Device:C_Small")
-		(at 219.71 149.86 0)
+		(lib_id "Connector:Conn_ARM_SWD_TagConnect_TC2030-NL")
+		(at 113.03 161.29 0)
 		(unit 1)
 		(body_style 1)
 		(exclude_from_sim no)
-		(in_bom yes)
+		(in_bom no)
 		(on_board yes)
 		(in_pos_files yes)
 		(dnp no)
 		(fields_autoplaced yes)
-		(property "Reference" "C5"
-			(at 222.25 148.5962 0)
+		(property "Reference" "J3"
+			(at 106.68 160.0199 0)
 			(show_name no)
 			(do_not_autoplace no)
@@
 					(size 1.27 1.27)
 				)
-				(justify left)
+				(justify right)
 			)
 		)
-		(property "Value" "4.7uF - Eth Reference Cap"
-			(at 222.25 151.1363 0)
+		(property "Value" "Conn_ARM_SWD_TagConnect_TC2030-NL"
+			(at 106.68 162.5599 0)
 			(show_name no)
 			(do_not_autoplace no)
 			(effects
 				(font
-					(size 0.8128 0.8128)
+					(size 1.27 1.27)
 				)
-				(justify left)
+				(justify right)
 			)
 		)
-		(property "Footprint" "Capacitor_SMD:C_0201_0603Metric"
-			(at 219.71 149.86 0)
+		(property "Footprint" "Connector:Tag-Connect_TC2030-IDC-NL_2x03_P1.27mm_Vertical"
+			(at 113.03 179.07 0)
 			(hide yes)
 			(show_name no)
@@
 			)
 		)
-		(property "Datasheet" ""
-			(at 219.71 149.86 0)
+		(property "Datasheet" "https://www.tag-connect.com/wp-content/uploads/bsk-pdf-manager/TC2030-CTX_1.pdf"
+			(at 113.03 176.53 0)
 			(hide yes)
 			(show_name no)
@@
 			)
 		)
-		(property "Description" "Unpolarized capacitor, small symbol"
-			(at 219.71 149.86 0)
+		(property "Description" "Tag-Connect ARM Cortex SWD JTAG connector, 6 pin, no legs"
+			(at 113.03 161.29 0)
 			(hide yes)
 			(show_name no)
@@
 			)
 		)
-		(pin "2"
+		(pin "5"
 		)
 		(pin "1"
 		)
+		(pin "3"
+		)
+		(pin "6"
+		)
+		(pin "4"
+		)
+		(pin "2"
+		)
 		(instances
 			(project "48VERelay"
 				(path "/2d740e7a-a48e-41b8-b74e-ca0ab277f7d9/856446f6-474b-446a-aa46-e1d1fc2a9600"
-					(reference "C5")
+					(reference "J3")
 					(unit 1)
 				)
@@
 			)
 		)
-		(property "Footprint" "Resistor_SMD:R_0201_0603Metric"
+		(property "Footprint" "Capacitor_SMD:C_0201_0603Metric"
 			(at 233.68 90.17 0)
 			(hide yes)
@@
 					(unit 1)
 				)
-			)
-		)
-	)
-	(symbol
-		(lib_id "power:+3V3")
-		(at 62.23 40.64 0)
-		(unit 1)
-		(body_style 1)
-		(exclude_from_sim no)
-		(in_bom yes)
-		(on_board yes)
-		(in_pos_files yes)
-		(dnp no)
-		(property "Reference" "#PWR061"
-			(at 62.23 44.45 0)
-			(hide yes)
-			(show_name no)
-			(do_not_autoplace no)
-			(effects
-				(font
-					(size 1.27 1.27)
-				)
-			)
-		)
-		(property "Value" "+3V3 MCU"
-			(at 61.722 37.338 0)
-			(show_name no)
-			(do_not_autoplace no)
-			(effects
-				(font
-					(size 1.27 1.27)
-				)
-			)
-		)
-		(property "Footprint" ""
-			(at 62.23 40.64 0)
-			(hide yes)
-			(show_name no)
-			(do_not_autoplace no)
-			(effects
-				(font
-					(size 1.27 1.27)
-				)
-			)
-		)
-		(property "Datasheet" ""
-			(at 62.23 40.64 0)
-			(hide yes)
-			(show_name no)
-			(do_not_autoplace no)
-			(effects
-				(font
-					(size 1.27 1.27)
-				)
-			)
-		)
-		(property "Description" "Power symbol creates a global label with name \"+3V3\""
-			(at 62.23 40.64 0)
-			(hide yes)
-			(show_name no)
-			(do_not_autoplace no)
-			(effects
-				(font
-					(size 1.27 1.27)
-				)
-			)
-		)
-		(pin "1"
-		)
-		(instances
-			(project "48VERelay"
-				(path "/2d740e7a-a48e-41b8-b74e-ca0ab277f7d9/856446f6-474b-446a-aa46-e1d1fc2a9600"
-					(reference "#PWR061")
-					(unit 1)
-				)
