File: RelatBoard/48VRelay/48VERelay/_restore_backup_2026-07-12T01-02-18-571/48VERelay.kicad_pcb (KiCad board)
At the start: 4 copper layers, 120 x 90 mm, 103 parts, among them J1 12, J10 Screw_Terminal_01x03, J11 Screw_Terminal_01x03, J12 Screw_Terminal_01x03, J13 Screw_Terminal_01x03, J14 Screw_Terminal_01x03, J2 RJ45_Hanrun_HR911105A_Horizon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, J4 TC2050, K10 G2RL-1-E, K11 G2RL-1-E, K12 G2RL-1-E, K13 G2RL-1-E, K14 G2RL-1-E, U1 ESP32-WROOM-32UE, U10 TLV1117LV33DCYR, U2 ULN2803A, U3 W5500, U4 3A 32V, U5 TPS630701RNMR, U7 TVS1800DRVR, U9 TLV1117LV33DCYR, Y2 ABM3C-25.000MHZ-D4Y-T

Commit message: Route ethernet
Parts:
- removed +3V3 MCU: TestPoint_Pad_D1.0mm, TestPoint:TestPoint_Pad_D1.0mm
- removed J4: TC2050, Connector:Tag-Connect_TC2050-IDC-NL_2x05_P1.27mm_Vertical
- added J3: Conn_ARM_SWD_TagConnect_TC2030-NL, Connector:Tag-Connect_TC2030-IDC-NL_2x03_P1.27mm_Vertical, F.Cu at (64.3, 162.6)
- R19: footprint Resistor_SMD:R_0201_0603Metric -> Capacitor_SMD:C_0201_0603Metric
- R21: footprint Resistor_SMD:R_0402_1005Metric -> Resistor_SMD:R_0603_1608Metric
- R22: footprint Resistor_SMD:R_0201_0603Metric -> Resistor_SMD:R_0603_1608Metric
- moved R19 35.5 mm to (42.9, 83.6)
- moved C6 32.9 mm to (45.2, 82.2), turned to 90 degrees
- moved R20 26.9 mm to (46.0, 84.7), turned to 90 degrees
- moved C20 24.0 mm to (47.5, 93.0)
- moved D6 23.9 mm to (56.6, 121.5)
- moved R29 23.9 mm to (60.5, 120.5), turned to 0 degrees
- moved C19 15.8 mm to (47.2, 97.2), turned to 0 degrees
- moved R22 14.7 mm to (47.8, 95.0)
- moved R18 14.2 mm to (43.8, 85.6), turned to 90 degrees
- moved R21 13.6 mm to (45.2, 88.5)
- moved C17 11.9 mm to (45.3, 92.6), turned to 0 degrees
- moved R7 8.00 mm to (41.5, 77.5)
- moved R8 8.00 mm to (43.0, 77.5)
- moved J2 2.19 mm to (58.9, 105.8)
- moved R15 2.19 mm to (46.8, 119.8)
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Routing:
- net /MCU/TX_N: track 11.0 -> 0.00 mm
- net +5V: track 37.3 -> 26.3 mm
- net /MCU/TX_P: track 10.8 -> 0.00 mm
- net /MCU/RX_N: track 7.19 -> 0.00 mm
- net /MCU/RX_P: track 7.01 -> 0.00 mm
